File: CL-232.kicad_pcb (KiCad board)
At the start: 2 copper layers, 100 x 80 mm, 42 parts, among them J1 Conn_01x06, J2 Screw_Terminal_01x10, J3 Barrel_Jack_Switch, J4 DE9_Socket, Q1 2N3904, Q2 2N3904, Q3 2N3904, Q4 2N3906, Q5 2N3904, U1 6N135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

Commit message: 2025-12-30 21:43
Parts:
- added D4: 1N4001, Diode_THT:D_DO-41_SOD81_P2.54mm_Vertical_AnodeUp, F.Cu at (97.3, 166.4)
- added J5: DB25_Socket, Connector_Dsub:DSUB-25_Socket_EdgeMount_P2.77mm, F.Cu at (78.7, 101.6)
- added J6: Conn_01x03, Connector_PinHeader_2.54mm:PinHeader_1x03_P2.54mm_Vertical, F.Cu at (92.7, 166.4)
- J4: value DE9_Socket -> DE9_Socket_MountingHoles
- moved C1 191.0 mm to (221.2, 96.3)
- moved C2 191.0 mm to (221.2, 100.4)
- moved C3 191.0 mm to (221.2, 104.4)
- moved C4 191.0 mm to (248.7, 87.8)
- moved C5 191.0 mm to (248.7, 91.9)
- moved C6 191.0 mm to (221.2, 108.5)
- moved C7 191.0 mm to (221.2, 112.5)
- moved C8 191.0 mm to (221.2, 116.6)
- moved C9 191.0 mm to (221.2, 120.6)
- moved D1 191.0 mm to (227.8, 61.5)
- moved D2 191.0 mm to (227.8, 65.0)
- moved D3 191.0 mm to (227.8, 68.6)
- moved J1 191.0 mm to (257.0, 109.2)
- moved Q1 191.0 mm to (239.4, 110.5)
- moved Q2 191.0 mm to (239.4, 116.6)
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Connections:
- net Net-(U4-R2IN) renamed TXRS
- net Net-(U4-T2OUT) renamed RXRS
- J3 pad 1: +12V -> Net-(D4-A)
- J4 pad 0: (no net) -> unconnected-(J4-PAD-Pad0)

Commit message: 2025-12-31
Parts:
- removed R10, R11, R12, R13: 240R, Resistor_THT:R_Axial_DIN0207_L6.3mm_D2.5mm_P10.16mm_Horizontal
- added J7: Conn_01x01, Connector_PinHeader_2.54mm:PinHeader_1x01_P2.54mm_Vertical, F.Cu at (88.9, 78.7)
- D4: footprint Diode_THT:D_DO-41_SOD81_P2.54mm_Vertical_AnodeUp -> Diode_THT:D_DO-41_SOD81_P10.16mm_Horizontal
- J2: footprint TerminalBlock_Phoenix:TerminalBlock_Phoenix_MPT-0,5-10-2.54_1x10_P2.54mm_Horizontal -> TerminalBlock_Phoenix:TerminalBlock_Phoenix_MPT-0,5-6-2.54_1x06_P2.54mm_Horizontal
- J6: footprint Connector_PinHeader_2.54mm:PinHeader_1x03_P2.54mm_Vertical -> Connector_PinHeader_2.54mm:PinHeader_1x03_P2.54mm_Horizontal
- Q3, Q5: footprint Package_TO_SOT_THT:TO-92_Inline -> Package_TO_SOT_THT:TO-92_HandSolder
- moved J1 144.6 mm to (113.0, 96.5)
- moved Q5 135.1 mm to (121.9, 115.6), turned to -90 degrees
- moved U4 128.8 mm to (99.1, 91.4)
- moved C6 126.9 mm to (95.2, 92.8), turned to -90 degrees
- moved C7 126.7 mm to (95.2, 99.1), turned to -90 degrees
- moved C5 124.7 mm to (124.5, 81.3), turned to -90 degrees
- moved C3 124.4 mm to (110.5, 161.3)
- moved C8 123.4 mm to (101.6, 86.4), turned to 180 degrees
- moved C9 122.0 mm to (104.2, 86.4)
- moved Q4 120.7 mm to (121.9, 95.2), turned to 90 degrees
- moved R8 117.3 mm to (106.7, 157.5)
- moved U1 117.1 mm to (129.5, 92.7)
- moved J6 115.3 mm to (167.6, 78.7)
- moved C4 109.2 mm to (139.7, 81.3), turned to -90 degrees
- moved D4 103.7 mm to (160.0, 83.8), turned to -90 degrees
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Connections:
- D4 pad 2: Net-(D4-A) -> ext-pwd
- J2 pad 1: Net-(D1-A) -> ext-pwd
- J2 pad 2: Net-(J2-Pin_2) -> GNDREF
- J2 pad 3: Net-(D3-K) -> Net-(D1-A)
- J2 pad 4: Net-(D3-A) -> Net-(J2-Pin_4)
- J2 pad 5: Net-(J2-Pin_5) -> Net-(D3-K)
- J2 pad 6: Net-(J2-Pin_6) -> Net-(D3-A)
- J3 pad 1: Net-(D4-A) -> ext-pwd
- Q2 pad 1: Net-(J2-Pin_2) -> Net-(J2-Pin_4)
- R1 pad 2: Net-(J2-Pin_2) -> Net-(J2-Pin_4)
- U1 pad 5: Net-(J2-Pin_2) -> Net-(J2-Pin_4)
Routing:
- net Net-(J6-Pin_1): track 0.00 -> 105.2 mm
- net +5V: track 0.00 -> 76.4 mm
- net Net-(D1-A): track 0.00 -> 49.7 mm
- net Net-(J2-Pin_4): track 0.00 -> 47.8 mm
- net Net-(D3-K): track 0.00 -> 44.6 mm
- net RXRS: track 0.00 -> 44.4 mm
- net TXRS: track 0.00 -> 42.8 mm
- net +12V: track 0.00 -> 33.0 mm
- net RX: track 0.00 -> 31.3 mm
- net Net-(U4-VS-): track 0.00 -> 21.2 mm
- net Net-(D3-A): track 0.00 -> 19.7 mm
- net ext-pwd: track 0.00 -> 19.0 mm
- net Net-(Q3-B): track 0.00 -> 17.2 mm
- net Net-(Q1-B): track 0.00 -> 16.0 mm
- net Net-(R4-Pad2): track 0.00 -> 14.7 mm
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- added copper zone on B.Cu, net (none)
- added copper zone on F.Cu, net (none)

Commit message: First Draft
Parts:
- J2: value Screw_Terminal_01x10 -> Screw_Terminal
- J4: value DE9_Socket_MountingHoles -> DE9_Socket
- moved R8 41.6 mm to (128.3, 121.9), turned to 180 degrees
- moved C3 38.8 mm to (124.5, 125.1), turned to 180 degrees
Connections:
- net +12V renamed Net-(J6-Pin_2)
- net Net-(J6-Pin_1) renamed Ami12V
Routing:
- net GNDREF: track 12.1 -> 38.9 mm
- net Net-(Q5-B): track 0.00 -> 19.3 mm
- net RX: track 31.3 -> 42.8 mm
- net Net-(C2-Pad1): track 11.5 -> 21.7 mm
- added copper zone on B.Cu, net GNDREF

Commit message: First revision is done.
Parts:
- added C10: 1µF, Capacitor_THT:C_Disc_D5.0mm_W2.5mm_P5.00mm, F.Cu at (111.7, 83.8)
- added J10: Conn_01x01, Connector_PinHeader_2.54mm:PinHeader_1x01_P2.54mm_Vertical, F.Cu at (120.7, 88.9)
- added J11: Conn_01x01, Connector_PinHeader_2.54mm:PinHeader_1x01_P2.54mm_Vertical, F.Cu at (130.8, 88.9)
- added J8: Conn_01x01, Connector_PinHeader_2.54mm:PinHeader_1x01_P2.54mm_Vertical, F.Cu at (106.7, 87.6)
- added J9: Conn_01x01, Connector_PinHeader_2.54mm:PinHeader_1x01_P2.54mm_Vertical, F.Cu at (111.8, 87.6)
- moved C9 4.53 mm to (100.9, 83.2), turned to 180 degrees
- moved C8 0.62 mm to (100.9, 86.4)
Connections:
- J4 pad 0: unconnected-(J4-PAD-Pad0) -> GNDREF
Routing:
- net GNDREF: track 38.9 -> 51.0 mm
- net Net-(U4-VS-): track 21.2 -> 24.6 mm
- net +5V: track 76.4 -> 75.8 mm
- added copper zone on F.Cu, net GNDREF

Commit message: More slime line
Parts:
- moved J6 18.9 mm to (149.9, 85.1), turned to 90 degrees
- moved H1 12.7 mm to (172.7, 124.5)
- moved H2 12.7 mm to (81.3, 124.5)
- moved H3 12.7 mm to (172.7, 78.7)
- moved H4 12.7 mm to (81.3, 78.7)
Routing:
- net Ami12V: track 105.2 -> 92.6 mm
- net Net-(J6-Pin_2): track 33.0 -> 24.9 mm
- net Net-(D4-K): track 7.62 -> 5.75 mm
- removed copper zone on B.Cu, net (none)
- removed copper zone on F.Cu, net (none)
Other:
- board size 100 x 80 mm -> 101 x 55.9 mm

Commit message: Version 0.2
Parts:
- removed J2: Screw_Terminal, TerminalBlock_Phoenix:TerminalBlock_Phoenix_MPT-0,5-6-2.54_1x06_P2.54mm_Horizontal
- added J12: Conn_01x06, Connector_Phoenix_MC_HighVoltage:PhoenixContact_MC_1,5_6-G-5.08_1x06_P5.08mm_Horizontal, F.Cu at (172.7, 114.3)
- moved D1 17.0 mm to (166.4, 91.4), turned to -90 degrees
- moved D4 9.16 mm to (154.9, 76.2)
- moved J3 7.63 mm to (163.8, 86.4), turned to -90 degrees
- moved Q1 6.35 mm to (151.1, 101.6)
- moved Q2 6.35 mm to (157.5, 101.6)
- moved D2 6.35 mm to (162.6, 99.1), turned to 90 degrees
- moved R2 6.35 mm to (158.8, 95.2)
- moved J6 5.08 mm to (144.8, 85.1)
- moved R1 4.85 mm to (145.1, 95.2)
- moved D3 2.54 mm to (166.4, 109.2)
- moved Q3 2.54 mm to (161.3, 114.3)
- moved R3 2.54 mm to (151.1, 118.1)
- moved U2 2.54 mm to (147.3, 118.1)
Routing:
- net GNDREF: track 51.0 -> 34.4 mm
- net Net-(D1-A): track 49.7 -> 40.7 mm
- net Net-(D4-K): track 5.75 -> 13.4 mm
- net Net-(D1-K): track 8.97 -> 3.81 mm
- net Net-(J6-Pin_2): track 24.9 -> 19.8 mm
- net Ami12V: track 92.6 -> 87.5 mm
- net Net-(D3-A): track 19.7 -> 16.6 mm
- net Net-(R6-Pad1): track 5.75 -> 8.29 mm
- net Net-(Q1-B): track 16.0 -> 17.9 mm
- net Net-(J12-Pin_3): track 47.8 -> 46.2 mm
- net Net-(C1-Pad2): track 6.41 -> 7.98 mm
- net Net-(C2-Pad1): track 21.7 -> 23.0 mm
- net ext-pwd: track 19.0 -> 19.7 mm
- net Net-(U4-VS-): track 24.6 -> 25.2 mm
