File: CL-232.kicad_pcb (KiCad board)
At the start: 2 copper layers, 101 x 55.9 mm, 47 parts, among them J1 Conn_01x06, J10 Conn_01x01, J11 Conn_01x01, J12 Conn_01x06, J3 Barrel_Jack_Switch, J4 DE9_Socket, J5 DB25_Socket, J6 Conn_01x03, J7 Conn_01x01, J8 Conn_01x01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

Commit message: Version 0.3
Parts:
- removed J7: Conn_01x01, Connector_PinHeader_2.54mm:PinHeader_1x01_P2.54mm_Vertical
- added D5: 1N4001, Diode_THT:D_DO-41_SOD81_P10.16mm_Horizontal, F.Cu at (99.1, 78.7)
Connections:
- J6 pad 1: Ami12V -> Net-(D5-K)
Routing:
- net Ami12V: track 87.5 -> 25.9 mm
- net Net-(D5-K): track 0.00 -> 51.5 mm

Commit message: Version 0.4
Parts:
- removed J10, J11, J8, J9: Conn_01x01, Connector_PinHeader_2.54mm:PinHeader_1x01_P2.54mm_Vertical
- added R10: 0R, Resistor_THT:R_Axial_DIN0204_L3.6mm_D1.6mm_P5.08mm_Horizontal, F.Cu at (127.0, 100.3)
- U3: footprint Package_TO_SOT_THT:TO-220-3_Vertical -> Package_TO_SOT_THT:TO-220F-3_Horizontal_TabDown
- moved C5 26.6 mm to (124.5, 107.9), turned to 90 degrees
- moved R4 23.4 mm to (132.1, 114.3), turned to 90 degrees
- moved C4 21.7 mm to (118.1, 78.8)
- moved U3 12.7 mm to (121.9, 81.3), turned to -90 degrees
- moved C10 4.02 mm to (110.5, 87.6)
- moved D4 1.27 mm to (153.7, 76.2)
- moved J6 1.27 mm to (143.5, 85.1)
- moved D5 1.27 mm to (99.1, 77.5)
- turned C2 to -90 degrees
Routing:
- net Net-(J6-Pin_2): track 19.8 -> 37.0 mm
- net GNDREF: track 34.4 -> 19.2 mm
- net +5V: track 75.8 -> 62.5 mm
- net Net-(D5-K): track 51.5 -> 56.0 mm
- net Net-(R4-Pad2): track 14.7 -> 10.8 mm
- net ext-pwd: track 19.7 -> 21.0 mm
- net Ami12V: track 25.9 -> 27.2 mm
Other:
- board text added: "+5V"
- board text added: "5v Logic"
- board text added: "Amiga ↑ Power Diode"
- board text added: "Current Loop"
- board text added: "GND"
- board text added: "Power"
- board text added: "R+"
- board text added: "R-"
- board text added: "RS232"
- board text added: "RX"
- board text added: "T+"
- board text added: "T-"
- board text added: "TX"
