File: CL-232.kicad_sch (KiCad schematic)
At the start: 29 parts, among them J1 Conn_01x06, J2 Screw_Terminal_01x10, Q1 2N3904, Q2 2N3904, Q3 2N3904, Q4 2N3906, Q5 2N3904, U1 6N135, U2 4N35, U3 LM7805_TO220

Commit message: Upload files to "/"
Parts:
- added C4, C5: 1µF, Capacitor_THT:C_Disc_D5.0mm_W2.5mm_P5.00mm, symbol Device:C
- added C6, C7, C8, C9: 100nF, Capacitor_THT:C_Disc_D5.0mm_W2.5mm_P2.50mm, symbol Device:C
- added H1, H2, H3, H4: MountingHole, MountingHole:MountingHole_3.2mm_M3_ISO14580, symbol Mechanical:MountingHole
- added J3: Barrel_Jack_Switch, Connector_BarrelJack:BarrelJack_Horizontal, symbol Connector:Barrel_Jack_Switch
- added J4: DE9_Socket, Connector_Dsub:DSUB-9_Socket_Horizontal_P2.77x2.84mm_EdgePinOffset4.94mm_Housed_MountingHolesOffset4.94mm, symbol Connector:DE9_Socket
- added U4: MAX3232, Package_DIP:DIP-16_W7.62mm_Socket_LongPads, symbol Interface_UART:MAX3232
Connections:
- net +12V: now also U3.1 (VI), C4.1, J3.1
- net +5V: now also U3.3 (VO), C5.1, U4.16 (VCC)
- net GNDREF: now also U3.2 (GND), C4.2, C5.2, C8.2, C9.2, J3.2, J3.3, J4.5, U4.15 (GND)
- net RX: now also U4.10 (T2IN)
- net TX: now also U4.9 (R2OUT)
- new net: C6.1, U4.1 (C1+)
- new net: C8.1, U4.2 (VS+)
- new net: C6.2, U4.3 (C1-)
- new net: C7.1, U4.4 (C2+)
- new net: C7.2, U4.5 (C2-)
- new net: C9.1, U4.6 (VS-)
- new net: J4.2, U4.7 (T2OUT)
- new net: J4.3, U4.8 (R2IN)
Other:
- moved on the sheet: U3

Commit message: 2025-12-30 21:43
Parts:
- removed J4: DE9_Socket, Connector_Dsub:DSUB-9_Socket_Horizontal_P2.77x2.84mm_EdgePinOffset4.94mm_Housed_MountingHolesOffset4.94mm, symbol Connector:DE9_Socket
- added D4: 1N4001, Diode_THT:D_DO-41_SOD81_P2.54mm_Vertical_AnodeUp, symbol Diode:1N4001
- added J4: DE9_Socket_MountingHoles, Connector_Dsub:DSUB-9_Socket_Horizontal_P2.77x2.84mm_EdgePinOffset4.94mm_Housed_MountingHolesOffset4.94mm, symbol Connector:DE9_Socket_MountingHoles
- added J5: DB25_Socket, Connector_Dsub:DSUB-25_Socket_EdgeMount_P2.77mm, symbol Connector:DB25_Socket
- added J6: Conn_01x03, Connector_PinHeader_2.54mm:PinHeader_1x03_P2.54mm_Vertical, symbol Connector_Generic:Conn_01x03
Connections:
- net +12V: now also J6.2 (Pin_2); no longer J3.1
- net GNDREF: now also J4.5, J5.7
- net RXRS: now reaches U4.7 (T2OUT)
- net RXRS: now also J4.2, J5.3
- net TXRS: now reaches U4.8 (R2IN)
- net TXRS: now also J4.3, J5.2
- new net: D4.2 (A), J3.1
- new net: J5.9, J6.1 (Pin_1)
- new net: D4.1 (K), J6.3 (Pin_3)
Other:
- moved on the sheet: J3

Commit message: 2025-12-31
Parts:
- removed R10, R11, R12, R13: 240R, Resistor_THT:R_Axial_DIN0207_L6.3mm_D2.5mm_P10.16mm_Horizontal, symbol Device:R
- added J7: Conn_01x01, Connector_PinHeader_2.54mm:PinHeader_1x01_P2.54mm_Vertical, symbol Connector_Generic:Conn_01x01
- D4: footprint Diode_THT:D_DO-41_SOD81_P2.54mm_Vertical_AnodeUp -> Diode_THT:D_DO-41_SOD81_P10.16mm_Horizontal
- J2: footprint TerminalBlock_Phoenix:TerminalBlock_Phoenix_MPT-0,5-10-2.54_1x10_P2.54mm_Horizontal -> TerminalBlock_Phoenix:TerminalBlock_Phoenix_MPT-0,5-6-2.54_1x06_P2.54mm_Horizontal; symbol Connector:Screw_Terminal_01x10 -> Connector:Screw_Terminal_01x06
- J6: footprint Connector_PinHeader_2.54mm:PinHeader_1x03_P2.54mm_Vertical -> Connector_PinHeader_2.54mm:PinHeader_1x03_P2.54mm_Horizontal
- Q3, Q5: footprint Package_TO_SOT_THT:TO-92_Inline -> Package_TO_SOT_THT:TO-92_HandSolder
Connections:
- net +12V: no longer J2.8 (Pin_8)
- net GNDREF: now also J2.2 (Pin_2); no longer J2.10 (Pin_10), J2.9 (Pin_9)
- net at C1.1, D1.2 (A), R2.1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: now also J2.3 (Pin_3); no longer J2.1 (Pin_1)
- net at Q2.1 (E), R1.2, U1.5: now also J2.4 (Pin_4); no longer J2.2 (Pin_2)
- net at D3.1 (K), Q3.3 (C), U2.1: now also J2.5 (Pin_5); no longer J2.3 (Pin_3)
- net at D3.2 (A), Q3.1 (E), R3.2: now also J2.6 (Pin_6); no longer J2.4 (Pin_4)
- net ext-pwd: now reaches D4.2 (A), J3.1
- net ext-pwd: now also J2.1 (Pin_1)
- net at J5.9, J6.1 (Pin_1): now also J7.1 (Pin_1)
Other:
- moved on the sheet: J3

Commit message: First Draft
Parts:
- J2: value Screw_Terminal_01x10 -> Screw_Terminal
- J4: value DE9_Socket_MountingHoles -> DE9_Socket
Connections:
- net GNDREF: now also J4.0 (PAD)
- net Ami12V: now reaches J5.9, J6.1 (Pin_1), J7.1 (Pin_1)
- net +12V: no longer names the net of C4.1, J6.2 (Pin_2), U3.1 (VI)
Other:
- moved on the sheet: C1, C2, C3, C4, C5, C6, C7, C8, C9, D1, D2, D3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

Commit message: First revision is done.
Parts:
- added C10: 1µF, Capacitor_THT:C_Disc_D5.0mm_W2.5mm_P5.00mm, symbol Device:C
- added J10, J11, J8, J9: Conn_01x01, Connector_PinHeader_2.54mm:PinHeader_1x01_P2.54mm_Vertical, symbol Connector_Generic:Conn_01x01
Connections:
- net +5V: now also C10.1
- net GNDREF: now also C10.2, J10.1 (Pin_1), J11.1 (Pin_1), J8.1 (Pin_1), J9.1 (Pin_1)
Other:
- note added: "Power"
- note added: "RS232 <-> TTL232"
- note added: "USB <-> TTL232"
- moved on the sheet: C4, C5, D4, J1, J3, J6, U3

Commit message: Version 0.2
Parts:
- removed J2: Screw_Terminal, TerminalBlock_Phoenix:TerminalBlock_Phoenix_MPT-0,5-6-2.54_1x06_P2.54mm_Horizontal, symbol Connector:Screw_Terminal_01x06
- added J12: Conn_01x06, Connector_Phoenix_MC_HighVoltage:PhoenixContact_MC_1,5_6-G-5.08_1x06_P5.08mm_Horizontal, symbol Connector_Generic:Conn_01x06
Connections:
- net GNDREF: now also J12.5 (Pin_5)
- net ext-pwd: now also J12.6 (Pin_6)
- net at C1.1, D1.2 (A), R2.1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: now also J12.4 (Pin_4)
- net at Q2.1 (E), R1.2, U1.5: now also J12.3 (Pin_3)
- net at D3.1 (K), Q3.3 (C), U2.1: now also J12.2 (Pin_2)
- net at D3.2 (A), Q3.1 (E), R3.2: now also J12.1 (Pin_1)
Changed lines of the file:
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@@
 	(wire
 		(pts
-			(xy 269.24 66.04) (xy 262.89 66.04)
+			(xy 262.89 66.04) (xy 267.97 66.04)
 		)
 		(stroke
@@
 	(wire
 		(pts
-			(xy 269.24 63.5) (xy 266.7 63.5)
-		)
-		(stroke
-			(width 0)
-			(type default)
-		)
-	)
-	(wire
-		(pts
 			(xy 228.6 53.34) (xy 228.6 50.8)
 		)
@@
 	(wire
 		(pts
-			(xy 269.24 71.12) (xy 260.35 71.12)
-		)
-		(stroke
-			(width 0)
-			(type default)
-		)
-	)
-	(wire
-		(pts
 			(xy 194.31 40.64) (xy 196.85 40.64)
 		)
@@
 	(wire
 		(pts
-			(xy 266.7 60.96) (xy 269.24 60.96)
-		)
-		(stroke
-			(width 0)
-			(type default)
-		)
-	)
-	(wire
-		(pts
 			(xy 87.63 27.94) (xy 87.63 31.75)
 		)
@@
 	(wire
 		(pts
-			(xy 262.89 73.66) (xy 269.24 73.66)
-		)
-		(stroke
-			(width 0)
-			(type default)
-		)
-	)
-	(wire
-		(pts
 			(xy 48.26 29.21) (xy 48.26 31.75)
 		)
@@
 	(wire
 		(pts
+			(xy 266.7 63.5) (xy 267.97 63.5)
+		)
+		(stroke
+			(width 0)
+			(type default)
+		)
+	)
+	(wire
+		(pts
 			(xy 31.75 92.71) (xy 31.75 77.47)
 		)
@@
 	(wire
 		(pts
-			(xy 260.35 68.58) (xy 269.24 68.58)
+			(xy 154.94 185.42) (xy 154.94 187.96)
 		)
 		(stroke
@@
 	(wire
 		(pts
-			(xy 154.94 185.42) (xy 154.94 187.96)
+			(xy 143.51 187.96) (xy 147.32 187.96)
 		)
 		(stroke
@@
 	(wire
 		(pts
-			(xy 143.51 187.96) (xy 147.32 187.96)
+			(xy 217.17 35.56) (xy 217.17 53.34)
 		)
 		(stroke
@@
 	(wire
 		(pts
-			(xy 217.17 35.56) (xy 217.17 53.34)
+			(xy 38.1 168.91) (xy 41.91 168.91)
 		)
 		(stroke
@@
 	(wire
 		(pts
-			(xy 38.1 168.91) (xy 41.91 168.91)
+			(xy 191.77 95.25) (xy 191.77 102.87)
 		)
 		(stroke
@@
 	(wire
 		(pts
-			(xy 191.77 95.25) (xy 191.77 102.87)
+			(xy 266.7 60.96) (xy 267.97 60.96)
 		)
 		(stroke
@@
 	(wire
 		(pts
+			(xy 260.35 68.58) (xy 267.97 68.58)
+		)
+		(stroke
+			(width 0)
+			(type default)
+		)
+	)
+	(wire
+		(pts
 			(xy 64.77 27.94) (xy 64.77 34.29)
 		)
@@
 	(wire
 		(pts
+			(xy 260.35 71.12) (xy 267.97 71.12)
+		)
+		(stroke
+			(width 0)
+			(type default)
+		)
+	)
+	(wire
+		(pts
 			(xy 107.95 29.21) (xy 107.95 31.75)
 		)
@@
 	(wire
 		(pts
+			(xy 262.89 73.66) (xy 267.97 73.66)
+		)
+		(stroke
+			(width 0)
+			(type default)
+		)
+	)
+	(wire
+		(pts
 			(xy 63.5 184.15) (xy 63.5 186.69)
 		)
@@
 	)
 	(symbol
-		(lib_id "Connector:Screw_Terminal_01x06")
-		(at 274.32 66.04 0)
-		(unit 1)
-		(exclude_from_sim no)
-		(in_bom yes)
-		(on_board yes)
-		(dnp no)
-		(property "Reference" "J2"
-			(at 277.876 74.676 90)
-			(effects
-				(font
-					(size 1.27 1.27)
-				)
-				(justify left)
-			)
-		)
-		(property "Value" "Screw_Terminal"
-			(at 280.416 74.676 90)
-			(effects
-				(font
-					(size 1.27 1.27)
-				)
-				(justify left)
-			)
-		)
-		(property "Footprint" "TerminalBlock_Phoenix:TerminalBlock_Phoenix_MPT-0,5-6-2.54_1x06_P2.54mm_Horizontal"
-			(at 274.32 66.04 0)
-			(effects
-				(font
-					(size 1.27 1.27)
-				)
-				(hide yes)
-			)
-		)
-		(property "Datasheet" "~"
-			(at 274.32 66.04 0)
-			(effects
-				(font
-					(size 1.27 1.27)
-				)
-				(hide yes)
-			)
-		)
-		(property "Description" "Generic screw terminal, single row, 01x06, script generated (kicad-library-utils/schlib/autogen/connector/)"
-			(at 274.32 66.04 0)
-			(effects
-				(font
-					(size 1.27 1.27)
-				)
-				(hide yes)
-			)
-		)
-		(pin "5"
-		)
-		(pin "1"
-		)
-		(pin "2"
-		)
-		(pin "4"
-		)
-		(pin "6"
-		)
-		(pin "3"
-		)
-		(instances
-			(project ""
-				(path "/8d0d347e-691e-4cff-9d05-91a8158922bd"
-					(reference "J2")
-					(unit 1)
-				)
-			)
-		)
-	)
-	(symbol
 		(lib_id "power:+5V")
 		(at 62.23 118.11 0)
@@
 					(unit 1)
 				)
+			)
+		)
+	)
+	(symbol
+		(lib_id "Connector_Generic:Conn_01x06")
+		(at 273.05 68.58 0)
+		(mirror x)
+		(unit 1)
+		(exclude_from_sim no)
+		(in_bom yes)
+		(on_board yes)
+		(dnp no)
+		(property "Reference" "J12"
+			(at 275.59 68.5801 0)
+			(effects
+				(font
+					(size 1.27 1.27)
+				)
+				(justify left)
+			)
+		)
+		(property "Value" "Conn_01x06"
+			(at 275.59 66.0401 0)
+			(effects
+				(font
+					(size 1.27 1.27)
+				)
+				(justify left)
+			)
+		)
+		(property "Footprint" "Connector_Phoenix_MC_HighVoltage:PhoenixContact_MC_1,5_6-G-5.08_1x06_P5.08mm_Horizontal"
+			(at 273.05 68.58 0)
+			(effects
+				(font
+					(size 1.27 1.27)
+				)
+				(hide yes)
+			)
+		)
+		(property "Datasheet" "~"
+			(at 273.05 68.58 0)
+			(effects
+				(font
+					(size 1.27 1.27)
+				)
+				(hide yes)
+			)
+		)
+		(property "Description" "Generic connector, single row, 01x06, script generated (kicad-library-utils/schlib/autogen/connector/)"
+			(at 273.05 68.58 0)
+			(effects
+				(font
+					(size 1.27 1.27)
+				)
+				(hide yes)
+			)
+		)
+		(pin "1"
+		)
+		(pin "4"
+		)
+		(pin "3"
+		)
+		(pin "2"
+		)
+		(pin "5"
+		)
+		(pin "6"
+		)
+		(instances
+			(project ""
+				(path "/8d0d347e-691e-4cff-9d05-91a8158922bd"
+					(reference "J12")
+					(unit 1)
+				)

Commit message: Version 0.3
Parts:
- removed J7: Conn_01x01, Connector_PinHeader_2.54mm:PinHeader_1x01_P2.54mm_Vertical, symbol Connector_Generic:Conn_01x01
- added D5: 1N4001, Diode_THT:D_DO-41_SOD81_P10.16mm_Horizontal, symbol Diode:1N4001
Connections:
- net Ami12V: now also D5.2 (A); no longer J6.1 (Pin_1)
- new net: D5.1 (K), J6.1 (Pin_1)
Other:
- title: (none) -> Current Loop <-> RS232/TTL232
- moved on the sheet: C4, C5, U3

Commit message: Version 0.4
Parts:
- removed J10, J11, J8, J9: Conn_01x01, Connector_PinHeader_2.54mm:PinHeader_1x01_P2.54mm_Vertical, symbol Connector_Generic:Conn_01x01
- added R10: 0R, Resistor_THT:R_Axial_DIN0204_L3.6mm_D1.6mm_P5.08mm_Horizontal, symbol Device:R
- U3: footprint Package_TO_SOT_THT:TO-220-3_Vertical -> Package_TO_SOT_THT:TO-220F-3_Horizontal_TabDown
Connections:
- net GNDREF: now also R10.1, R10.2
